Commit message: Update

File: src/minibot_description/urdf/minibot.urdf.xacro (robot description, xacro)
@@ -23,10 +23,10 @@
     <parent link="base_footprint"/>
     <child link="base_link"/>
-    <origin xyz="0 0 0.03" rpy="0 0 0"/>
+    <origin xyz="0 0 0.04615" rpy="0 0 0"/>
   </joint>
   <link name="base_link">
     <visual>
       <geometry>
-        <box size="0.18 0.15 0.02"/>
+        <box size="0.27692 0.23077 0.03077"/>
       </geometry>
       <material name="charcoal"/>
@@ -34,11 +34,11 @@
     <collision>
       <geometry>
-        <box size="0.18 0.15 0.02"/>
-      </geometry>
-    </collision>
-    <inertial>
-      <mass value="1.0"/>
-      <origin xyz="0 0 0"/>
-      <inertia ixx="0.00191" ixy="0.0" ixz="0.0" iyy="0.00273" iyz="0.0" izz="0.00458"/>
+        <box size="0.27692 0.23077 0.03077"/>
+      </geometry>
+    </collision>
+    <inertial>
+      <mass value="3.6414"/>
+      <origin xyz="0 0 0"/>
+      <inertia ixx="0.01646" ixy="0.0" ixz="0.0" iyy="0.02353" iyz="0.0" izz="0.03947"/>
     </inertial>
   </link>
@@ -46,5 +46,5 @@
     <parent link="base_link"/>
     <child link="left_wheel"/>
-    <origin xyz="-0.04 0.09 0.0" rpy="-1.5708 0 0"/>
+    <origin xyz="-0.06154 0.13846 0.0" rpy="-1.5708 0 0"/>
     <axis xyz="0 0 1"/>
     <limit effort="20" velocity="20"/>
@@ -54,5 +54,5 @@
     <visual>
       <geometry>
-        <cylinder radius="0.03" length="0.025"/>
+        <cylinder radius="0.04615" length="0.03846"/>
       </geometry>
       <material name="terracotta"/>
@@ -60,11 +60,11 @@
     <collision>
       <geometry>
-        <cylinder radius="0.03" length="0.025"/>
-      </geometry>
-    </collision>
-    <inertial>
-      <mass value="0.20"/>
-      <origin xyz="0 0 0"/>
-      <inertia ixx="0.000055" ixy="0.0" ixz="0.0" iyy="0.000055" iyz="0.0" izz="0.00009"/>
+        <cylinder radius="0.04615" length="0.03846"/>
+      </geometry>
+    </collision>
+    <inertial>
+      <mass value="0.7283"/>
+      <origin xyz="0 0 0"/>
+      <inertia ixx="0.000474" ixy="0.0" ixz="0.0" iyy="0.000474" iyz="0.0" izz="0.000776"/>
     </inertial>
   </link>
@@ -72,5 +72,5 @@
     <parent link="base_link"/>
     <child link="right_wheel"/>
-    <origin xyz="-0.04 -0.09 0.0" rpy="-1.5708 0 0"/>
+    <origin xyz="-0.06154 -0.13846 0.0" rpy="-1.5708 0 0"/>
     <axis xyz="0 0 1"/>
     <limit effort="20" velocity="20"/>
@@ -80,5 +80,5 @@
     <visual>
       <geometry>
-        <cylinder radius="0.03" length="0.025"/>
+        <cylinder radius="0.04615" length="0.03846"/>
       </geometry>
       <material name="terracotta"/>
@@ -86,11 +86,11 @@
     <collision>
       <geometry>
-        <cylinder radius="0.03" length="0.025"/>
-      </geometry>
-    </collision>
-    <inertial>
-      <mass value="0.20"/>
-      <origin xyz="0 0 0"/>
-      <inertia ixx="0.000055" ixy="0.0" ixz="0.0" iyy="0.000055" iyz="0.0" izz="0.00009"/>
+        <cylinder radius="0.04615" length="0.03846"/>
+      </geometry>
+    </collision>
+    <inertial>
+      <mass value="0.7283"/>
+      <origin xyz="0 0 0"/>
+      <inertia ixx="0.000474" ixy="0.0" ixz="0.0" iyy="0.000474" iyz="0.0" izz="0.000776"/>
     </inertial>
   </link>
@@ -98,10 +98,10 @@
     <parent link="base_link"/>
     <child link="front_left_caster"/>
-    <origin xyz="0.06 0.055 -0.015" rpy="0 0 0"/>
+    <origin xyz="0.09231 0.08462 -0.02308" rpy="0 0 0"/>
   </joint>
   <link name="front_left_caster">
     <visual>
       <geometry>
-        <sphere radius="0.015"/>
+        <sphere radius="0.02308"/>
       </geometry>
       <material name="sand"/>
@@ -109,11 +109,11 @@
     <collision>
       <geometry>
-        <sphere radius="0.015"/>
-      </geometry>
-    </collision>
-    <inertial>
-      <mass value="0.04"/>
-      <origin xyz="0 0 0"/>
-      <inertia ixx="0.0000036" ixy="0.0" ixz="0.0" iyy="0.0000036" iyz="0.0" izz="0.0000036"/>
+        <sphere radius="0.02308"/>
+      </geometry>
+    </collision>
+    <inertial>
+      <mass value="0.1457"/>
+      <origin xyz="0 0 0"/>
+      <inertia ixx="0.000031" ixy="0.0" ixz="0.0" iyy="0.000031" iyz="0.0" izz="0.000031"/>
     </inertial>
   </link>
@@ -121,10 +121,10 @@
     <parent link="base_link"/>
     <child link="front_right_caster"/>
-    <origin xyz="0.06 -0.055 -0.015" rpy="0 0 0"/>
+    <origin xyz="0.09231 -0.08462 -0.02308" rpy="0 0 0"/>
   </joint>
   <link name="front_right_caster">
     <visual>
       <geometry>
-        <sphere radius="0.015"/>
+        <sphere radius="0.02308"/>
       </geometry>
       <material name="sand"/>
@@ -132,11 +132,11 @@
     <collision>
       <geometry>
-        <sphere radius="0.015"/>
-      </geometry>
-    </collision>
-    <inertial>
-      <mass value="0.04"/>
-      <origin xyz="0 0 0"/>
-      <inertia ixx="0.0000036" ixy="0.0" ixz="0.0" iyy="0.0000036" iyz="0.0" izz="0.0000036"/>
+        <sphere radius="0.02308"/>
+      </geometry>
+    </collision>
+    <inertial>
+      <mass value="0.1457"/>
+      <origin xyz="0 0 0"/>
+      <inertia ixx="0.000031" ixy="0.0" ixz="0.0" iyy="0.000031" iyz="0.0" izz="0.000031"/>
     </inertial>
   </link>
@@ -144,11 +144,10 @@
     <parent link="base_link"/>
     <child link="battery_link"/>
-    <origin xyz="0.0 0.0 0.025" rpy="0 0 0"/>
-  </joint>
-  <!-- FIX: removed stray <hold_joints> tag that was incorrectly placed inside this link's collision block -->
+    <origin xyz="0.0 0.0 0.03846" rpy="0 0 0"/>
+  </joint>
   <link name="battery_link">
     <visual>
       <geometry>
-        <box size="0.15 0.07 0.03"/>
+        <box size="0.23077 0.10769 0.04615"/>
       </geometry>
       <material name="muddy_brown"/>
@@ -156,11 +155,11 @@
     <collision>
       <geometry>
-        <box size="0.15 0.07 0.03"/>
-      </geometry>
-    </collision>
-    <inertial>
-      <mass value="0.6"/>
-      <origin xyz="0 0 0"/>
-      <inertia ixx="0.00029" ixy="0.0" ixz="0.0" iyy="0.00117" iyz="0.0" izz="0.00137"/>
+        <box size="0.23077 0.10769 0.04615"/>
+      </geometry>
+    </collision>
+    <inertial>
+      <mass value="2.1848"/>
+      <origin xyz="0 0 0"/>
+      <inertia ixx="0.00250" ixy="0.0" ixz="0.0" iyy="0.01008" iyz="0.0" izz="0.01181"/>
     </inertial>
   </link>
@@ -168,10 +167,10 @@
     <parent link="battery_link"/>
     <child link="orin_link"/>
-    <origin xyz="0.0 0.0 0.0475" rpy="0 0 0"/>
+    <origin xyz="0.0 0.0 0.07308" rpy="0 0 0"/>
   </joint>
   <link name="orin_link">
     <visual>
       <geometry>
-        <box size="0.105 0.105 0.065"/>
+        <box size="0.16154 0.16154 0.10000"/>
       </geometry>
       <material name="slate_blue"/>
@@ -179,11 +178,11 @@
     <collision>
       <geometry>
-        <box size="0.105 0.105 0.065"/>
-      </geometry>
-    </collision>
-    <inertial>
-      <mass value="0.7"/>
-      <origin xyz="0 0 0"/>
-      <inertia ixx="0.00089" ixy="0.0" ixz="0.0" iyy="0.00089" iyz="0.0" izz="0.00129"/>
+        <box size="0.16154 0.16154 0.10000"/>
+      </geometry>
+    </collision>
+    <inertial>
+      <mass value="2.5490"/>
+      <origin xyz="0 0 0"/>
+      <inertia ixx="0.00767" ixy="0.0" ixz="0.0" iyy="0.00767" iyz="0.0" izz="0.01112"/>
     </inertial>
   </link>
@@ -191,50 +190,50 @@
     <parent link="base_link"/>
     <child link="camera_rods_link"/>
-    <origin xyz="0.08 0.0 0.01" rpy="0 0 0"/>
+    <origin xyz="0.12308 0.0 0.01538" rpy="0 0 0"/>
   </joint>
   <link name="camera_rods_link">
     <visual>
-      <origin xyz="0.0 0.05 0.05" rpy="0 0 0"/>
-      <geometry>
-        <cylinder radius="0.004" length="0.10"/>
+      <origin xyz="0.0 0.07692 0.10192" rpy="0 0 0"/>
+      <geometry>
+        <cylinder radius="0.00615" length="0.20385"/>
       </geometry>
       <material name="charcoal"/>
     </visual>
     <visual>
-      <origin xyz="0.0 -0.05 0.05" rpy="0 0 0"/>
-      <geometry>
-        <cylinder radius="0.004" length="0.10"/>
+      <origin xyz="0.0 -0.07692 0.10192" rpy="0 0 0"/>
+      <geometry>
+        <cylinder radius="0.00615" length="0.20385"/>
       </geometry>
       <material name="charcoal"/>
     </visual>
     <visual>
-      <origin xyz="0.0 0.0 0.101" rpy="0 0 0"/>
-      <geometry>
-        <box size="0.02 0.12 0.002"/>
+      <origin xyz="0.0 0.0 0.20538" rpy="0 0 0"/>
+      <geometry>
+        <box size="0.03077 0.18462 0.00308"/>
       </geometry>
       <material name="charcoal"/>
     </visual>
     <collision>
-      <origin xyz="0.0 0.05 0.05" rpy="0 0 0"/>
-      <geometry>
-        <cylinder radius="0.004" length="0.10"/>
-      </geometry>
-    </collision>
-    <collision>
-      <origin xyz="0.0 -0.05 0.05" rpy="0 0 0"/>
-      <geometry>
-        <cylinder radius="0.004" length="0.10"/>
-      </geometry>
-    </collision>
-    <collision>
-      <origin xyz="0.0 0.0 0.101" rpy="0 0 0"/>
-      <geometry>
-        <box size="0.02 0.12 0.002"/>
-      </geometry>
-    </collision>
-    <inertial>
-      <mass value="0.05"/>
-      <origin xyz="0.0 0.0 0.06"/>
-      <inertia ixx="0.000046" ixy="0.0" ixz="0.0" iyy="0.000035" iyz="0.0" izz="0.000013"/>
+      <origin xyz="0.0 0.07692 0.10192" rpy="0 0 0"/>
+      <geometry>
+        <cylinder radius="0.00615" length="0.20385"/>
+      </geometry>
+    </collision>
+    <collision>
+      <origin xyz="0.0 -0.07692 0.10192" rpy="0 0 0"/>
+      <geometry>
+        <cylinder radius="0.00615" length="0.20385"/>
+      </geometry>
+    </collision>
+    <collision>
+      <origin xyz="0.0 0.0 0.20538" rpy="0 0 0"/>
+      <geometry>
+        <box size="0.03077 0.18462 0.00308"/>
+      </geometry>
+    </collision>
+    <inertial>
+      <mass value="0.1821"/>
+      <origin xyz="0.0 0.0 0.11731"/>
+      <inertia ixx="0.000396" ixy="0.0" ixz="0.0" iyy="0.000302" iyz="0.0" izz="0.000112"/>
     </inertial>
   </link>
@@ -242,10 +241,10 @@
     <parent link="camera_rods_link"/>
     <child link="zed2i_camera_link"/>
-    <origin xyz="0.01 0.0 0.1225" rpy="0 0 0"/>
+    <origin xyz="0.01538 0.0 0.23846" rpy="0 0 0"/>
   </joint>
   <link name="zed2i_camera_link">
     <visual>
       <geometry>
-        <box size="0.03 0.175 0.043"/>
+        <box size="0.04615 0.26923 0.06615"/>
       </geometry>
       <material name="matte_black"/>
@@ -253,11 +252,11 @@
     <collision>
       <geometry>
-        <box size="0.03 0.175 0.043"/>
-      </geometry>
-    </collision>
-    <inertial>
-      <mass value="0.16"/>
-      <origin xyz="0 0 0"/>
-      <inertia ixx="0.000433" ixy="0.0" ixz="0.0" iyy="0.000024" iyz="0.0" izz="0.000421"/>
+        <box size="0.04615 0.26923 0.06615"/>
+      </geometry>
+    </collision>
+    <inertial>
+      <mass value="0.5826"/>
+      <origin xyz="0 0 0"/>
+      <inertia ixx="0.003732" ixy="0.0" ixz="0.0" iyy="0.000207" iyz="0.0" izz="0.003628"/>
     </inertial>
   </link>
@@ -268,8 +267,6 @@
   </joint>
   <link name="camera_link_optical"/>
-  <!-- ==================== ROS2 CONTROL ==================== -->
   <ros2_control name="GazeboSystem" type="system">
     <hardware>
-      <!-- FIX: correct plugin name for gz_ros2_control on Humble/Fortress -->
       <plugin>gz_ros2_control/GazeboSimSystem</plugin>
     </hardware>
@@ -291,16 +288,4 @@
     </joint>
   </ros2_control>
-  <!-- ==================== GAZEBO PLUGIN ==================== -->
-  <!--
-    FIX 1: filename must be "gz_ros2_control-system" (no "lib" prefix, no ".so").
-    FIX 2: name attribute must use double-colon namespace syntax.
-    FIX 3: Added <robot_param> and <robot_param_node> so the plugin can find
-            the URDF on the ROS parameter server.
-    FIX 4: Removed the broken <ros><remapping> block. The cmd_vel remapping
-            is now done cleanly in the launch file via the controller spawner
-            or a standalone topic_tools/relay node.
-    FIX 5: Removed <hold_joints> — it belongs INSIDE the plugin tag, not
-            in a link. Set to false so wheels are free to rotate on spawn.
-  -->
   <gazebo>
     <plugin filename="gz_ros2_control-system"
@@ -312,5 +297,4 @@
     </plugin>
   </gazebo>
-  <!-- ==================== WHEEL FRICTION ==================== -->
   <gazebo reference="front_left_caster">
     <mu1>0.0</mu1>
@@ -329,5 +313,4 @@
     <mu2>1.0</mu2>
   </gazebo>
-  <!--SENSORS-->
   <gazebo reference="orin_link">
       <sensor name="minibot_imu" type="imu">
